Commit message: feat(firmware): update ESP32 firmware for new hardware
The robot wiring and firmware requirements changed: motors were
rewired to a TB6612FNG driver and new sensors (MPU6050 IMU,
single‑phase encoders, pan‑tilt servos) were added. Also resolve
micro-ROS build conflicts by upgrading PlatformIO and isolating the
build environment.

- Update GPIO pin mapping in firmware/include/config.h to match
  TB6612FNG wiring and avoid boot-sensitive pins
- Add LEDC channel defines to firmware/include/config.h to reserve
  PWM channels for motors, LiDAR motor, and servos
- Add encoder pin and constants to firmware/include/config.h to
  support single-phase wheel encoders for odometry
- Add MPU6050 I2C pins and IMU constants to firmware/include/config.h
  to enable IMU initialization and publishing
- Add servo pan/tilt pin and center constant to
  firmware/include/config.h
  to support pan-tilt control
- Update LiDAR motor and UART pin defines to firmware/include/config.h
  to match LDS02RR wiring
- Add micro_ros.meta to firmware to increase MTU and entity limits to
  support 360-point LaserScan messages
- Upgrade PlatformIO platform and add MPU6050/ESP32Servo libs in
  firmware/platformio.ini to build required libraries
- Add pre-build script (scripts/clean_ros_env.py) and
  pio_isolated_build.sh to isolate PlatformIO builds from host ROS2
  environment and prevent CMake package conflicts
- Update firmware/src/main.cpp and cam_main.cpp to initialize IMU,
  encoders, servos, LiDAR, and to parse AGENT_IP for micro-ROS transport
- Add odometry, IMU, joint_state, scan publishers and cmd_vel/servo_cmd
  subscribers in firmware to expose sensors and actuators to ROS2
- Add URDF pan-tilt and imu_link changes and robot_localization EKF
  config/launch to enable PC-side odom+IMU fusion and joint TFs
- Update Nav2 params and package.xml to use fused odometry topic
  (/odometry/filtered) for navigation
- Add openspec change archives and specs documenting requirements,
  tasks, and verification for the hardware and firmware updates

BREAKING CHANGE: Motor driver pin mapping changed from L298N to
TB6612FNG and PlatformIO platform upgraded to espressif32@6.13.0.
Developers must update firmware/include/config.h, refresh local
PlatformIO environments, and rebuild firmware in the isolated build
environment.

Signed-off-by: Nguyễn Ngọc Phú <ngocphunguyenabc@gmail.com>

File: src/slam_car_bringup/urdf/robot.urdf.xacro (robot description, xacro)
@@ -147,5 +147,36 @@
     <origin xyz="0 0 ${chassis_height/2 + lidar_height/2}" rpy="0 0 0"/>
   </joint>
-  <!-- ── Camera (ESP32-CAM) ─────────────────────────────────── -->
+  <!-- ── IMU (MPU6050) ─────────────────────────────────────── -->
+  <link name="imu_link"/>
+  <joint name="imu_joint" type="fixed">
+    <parent link="base_link"/>
+    <child link="imu_link"/>
+    <origin xyz="0 0 ${chassis_height/2}" rpy="0 0 0"/>
+  </joint>
+  <!-- ── Pan-Tilt Camera Mount (ESP32-CAM) ───────────────────── -->
+  <!-- Pan link (rotates around Z axis) -->
+  <link name="pan_link">
+    <visual>
+      <geometry>
+        <cylinder radius="0.01" length="0.02"/>
+      </geometry>
+      <material name="gray">
+        <color rgba="0.5 0.5 0.5 1.0"/>
+      </material>
+    </visual>
+    <inertial>
+      <mass value="0.02"/>
+      <inertia ixx="0.000001" ixy="0" ixz="0" iyy="0.000001" iyz="0" izz="0.000001"/>
+    </inertial>
+  </link>
+  <joint name="camera_pan_joint" type="revolute">
+    <parent link="base_link"/>
+    <child link="pan_link"/>
+    <origin xyz="${chassis_length/2} 0 ${chassis_height/4}" rpy="0 0 0"/>
+    <axis xyz="0 0 1"/>
+    <limit lower="${-pi/2}" upper="${pi/2}" effort="1.0" velocity="2.0"/>
+    <dynamics damping="0.01" friction="0.1"/>
+  </joint>
+  <!-- Camera link (rotates around Y axis for tilt) -->
   <link name="camera_link">
     <visual>
@@ -164,8 +195,11 @@
     <xacro:box_inertia m="${camera_mass}" x="${camera_size}" y="${camera_size}" z="${camera_size}"/>
   </link>
-  <joint name="camera_joint" type="fixed">
-    <parent link="base_link"/>
+  <joint name="camera_tilt_joint" type="revolute">
+    <parent link="pan_link"/>
     <child link="camera_link"/>
-    <origin xyz="${chassis_length/2} 0 ${chassis_height/4}" rpy="0 0 0"/>
+    <origin xyz="0 0 0.01" rpy="0 0 0"/>
+    <axis xyz="0 1 0"/>
+    <limit lower="${-pi/2}" upper="${pi/2}" effort="1.0" velocity="2.0"/>
+    <dynamics damping="0.01" friction="0.1"/>
   </joint>
   <!-- Camera optical frame (Z forward, X right, Y down — ROS convention) -->

Commit message: feat(ui): add unified dashboard with enrollment and tracking
Operators currently switch between multiple pages for SLAM, tracking, and
enrollment which fragments state and complicates live robot control. This
change introduces a single unified dashboard plus enrollment and person
tracking integration to improve operator flow, resilience, and target
management.

- Add unified dashboard route and UnifiedDashboard orchestrator to
  consolidate SLAM and tracking into a single operator workspace
- Add dashboard keyboard handler, mode controller, status bar, and
  reconnect overlay to provide global shortcuts, mode switching, telemetry,
  and recovery affordances
- Add adaptive viewport system (PrimaryViewport, PictureInPicture,
  MinimapOverlay, ViewportSwitcher) to present map/camera primary and
  secondary surfaces per active mode
- Add enrollment UI (Enrollment page, WebcamCapture, ScanOverlay,
  EnrollForm, PersonList, PersonCard, EnrollModal) to capture webcam
  frames and manage enrolled persons from the dashboard
- Add enrollment hook, Zustand stores, and services integration to call
  ROS2 enrollment services for add/remove/list/set/get target functionality
- Add person-tracking message types (BoundingBox2D, TrackedPerson,
  TrackedPersonArray, EnrolledPerson, EnrollmentStatus) and services
  (AddPerson, RemovePerson, ListPersons, SetTrackingTarget, GetTrackingTarget)
  to support robust body+face tracking and enrollment
- Add person tracking launch (person_tracking.launch.py) and replace
  legacy face-tracking launch with the new flow to orchestrate enrollment,
  tracker, controller, and rosbridge
- Update tracking UI (PersonOverlay, TrackingPanels, TrackingStatus) and
  add tests (vitest) for keyboard handling, viewport composition, and
  dashboard store behavior to verify control gating and layout rules
- Update development container Dockerfile to install ultralytics,
  insightface, onnxruntime and pre-download models; pin numpy<2 to avoid
  ABI incompatibilities with InsightFace wheels
- Add firmware improvements and build tooling (firmware/.env.example,
  load_env.py, platformio updates, pan-only servo changes, logger,
  safety updates) to support environment-driven builds and pan-only servo
- Add CI/dev tooling (vitest.config.ts, commitlint, lefthook, ruff,
  pyproject.toml) to enforce linting, commit message checks, and tests

BREAKING CHANGE: Deprecate legacy multi-page operator flow (/, /slam,
/tracking, /enrollment) in favor of /dashboard; replace /face_detections
(PoseArray) with /tracked_persons (TrackedPersonArray) and related ROS
interfaces; remove tilt servo support in firmware (pan-only servo).

Signed-off-by: Nguyễn Ngọc Phú <ngocphunguyenabc@gmail.com>

File: src/slam_car_bringup/urdf/robot.urdf.xacro (robot description, xacro)
@@ -154,6 +154,7 @@
     <origin xyz="0 0 ${chassis_height/2}" rpy="0 0 0"/>
   </joint>
-  <!-- ── Pan-Tilt Camera Mount (ESP32-CAM) ───────────────────── -->
+  <!-- ── Pan Camera Mount (ESP32-CAM) ─────────────────────────── -->
   <!-- Pan link (rotates around Z axis) -->
+  <!-- Note: Tilt servo removed per design decision (pan-only tracking) -->
   <link name="pan_link">
     <visual>
@@ -178,5 +179,5 @@
     <dynamics damping="0.01" friction="0.1"/>
   </joint>
-  <!-- Camera link (rotates around Y axis for tilt) -->
+  <!-- Camera link (attached directly to pan link — no tilt) -->
   <link name="camera_link">
     <visual>
@@ -195,11 +196,8 @@
     <xacro:box_inertia m="${camera_mass}" x="${camera_size}" y="${camera_size}" z="${camera_size}"/>
   </link>
-  <joint name="camera_tilt_joint" type="revolute">
+  <joint name="camera_mount_joint" type="fixed">
     <parent link="pan_link"/>
     <child link="camera_link"/>
     <origin xyz="0 0 0.01" rpy="0 0 0"/>
-    <axis xyz="0 1 0"/>
-    <limit lower="${-pi/2}" upper="${pi/2}" effort="1.0" velocity="2.0"/>
-    <dynamics damping="0.01" friction="0.1"/>
   </joint>
   <!-- Camera optical frame (Z forward, X right, Y down — ROS convention) -->
